File: tx_output.kicad_sch (KiCad schematic)
At the start: 0 parts

Commit message: More filter work. Add project title to drawings.
Other:
- company: (none) -> Steves Custom Computers
- title: (none) -> PLUTO RF Card Front-End
Changed lines of the file:
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@@
 (kicad_sch (version 20230121) (generator eeschema)
   (paper "A4")
+  (title_block
+    (title "PLUTO RF Card Front-End")
+    (rev " 001")
+    (company "Steves Custom Computers")
+  )
 )
