File: rx_output.kicad_sch (KiCad schematic)
At the start: 0 parts

Commit message: More filter work. Add project title to drawings.
Other:
- company: (none) -> Steves Custom Computers
- title: (none) -> PLUTO RF Card Front-End
Changed lines of the file:
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@@
 (kicad_sch (version 20230121) (generator eeschema)
   (paper "A4")
+  (title_block
+    (title "PLUTO RF Card Front-End")
+    (rev " 001")
+    (company "Steves Custom Computers")
+  )
 )

Commit message: Major restructure. Add power/control busses.
Parts:
- added J5: PCB.SMAFRA.HT, PCBSMAFRAHT, symbol Mouser:PCB.SMAFRA.HT
Connections:
- new net GND: J5.2, J5.3, J5.4, J5.5
- new net RX: J5.1
Other:
- title: PLUTO RF Card Front-End -> PLUTO RF Front-End Card
Changed lines of the file:
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@@
   (paper "A4")
   (title_block
-    (title "PLUTO RF Card Front-End")
+    (title "PLUTO RF Front-End Card")
     (rev " 001")
     (company "Steves Custom Computers")
   )
+  (junction (at 76.2 34.29) (diameter 0) (color 0 0 0 0)
+  )
+  (junction (at 41.91 36.83) (diameter 0) (color 0 0 0 0)
+  )
+  (junction (at 41.91 41.91) (diameter 0) (color 0 0 0 0)
+  )
+  (wire (pts (xy 27.94 31.75) (xy 49.53 31.75))
+    (stroke (width 0) (type default))
+  )
+  (wire (pts (xy 49.53 34.29) (xy 41.91 34.29))
+    (stroke (width 0) (type default))
+  )
+  (wire (pts (xy 41.91 41.91) (xy 41.91 46.99))
+    (stroke (width 0) (type default))
+  )
+  (wire (pts (xy 69.85 31.75) (xy 76.2 31.75))
+    (stroke (width 0) (type default))
+  )
+  (wire (pts (xy 76.2 31.75) (xy 76.2 34.29))
+    (stroke (width 0) (type default))
+  )
+  (wire (pts (xy 41.91 36.83) (xy 49.53 36.83))
+    (stroke (width 0) (type default))
+  )
+  (wire (pts (xy 76.2 41.91) (xy 41.91 41.91))
+    (stroke (width 0) (type default))
+  )
+  (wire (pts (xy 41.91 36.83) (xy 41.91 41.91))
+    (stroke (width 0) (type default))
+  )
+  (wire (pts (xy 76.2 34.29) (xy 76.2 41.91))
+    (stroke (width 0) (type default))
+  )
+  (wire (pts (xy 41.91 34.29) (xy 41.91 36.83))
+    (stroke (width 0) (type default))
+  )
+  (wire (pts (xy 69.85 34.29) (xy 76.2 34.29))
+    (stroke (width 0) (type default))
+  )
+  (hierarchical_label "RX" (shape input) (at 27.94 31.75 180) (fields_autoplaced)
+    (effects (font (size 1.27 1.27)) (justify right))
+  )
+  (symbol (lib_id "Mouser:PCB.SMAFRA.HT") (at 49.53 31.75 0) (unit 1)
+    (in_bom yes) (on_board yes) (dnp no) (fields_autoplaced)
+    (property "Reference" "J5" (at 59.69 24.13 0)
+      (effects (font (size 1.27 1.27)))
+    )
+    (property "Value" "PCB.SMAFRA.HT" (at 59.69 26.67 0)
+      (effects (font (size 1.27 1.27)))
+    )
+    (property "Footprint" "PCBSMAFRAHT" (at 66.04 126.67 0)
+      (effects (font (size 1.27 1.27)) (justify left top) hide)
+    )
+    (property "Datasheet" "" (at 66.04 226.67 0)
+      (effects (font (size 1.27 1.27)) (justify left top) hide)
+    )
+    (property "Height" "9" (at 66.04 426.67 0)
+      (effects (font (size 1.27 1.27)) (justify left top) hide)
+    )
+    (property "Mouser Part Number" "960-PCB.SMAFRA.HT" (at 66.04 526.67 0)
+      (effects (font (size 1.27 1.27)) (justify left top) hide)
+    )
+    (property "Mouser Price/Stock" "https://www.mouser.co.uk/ProductDetail/Taoglas/PCB.SMAFRA.HT?qs=RuW%2Fu%252BNMQmubIFYcN8w5Dw%3D%3D" (at 66.04 626.67 0)
+      (effects (font (size 1.27 1.27)) (justify left top) hide)
+    )
+    (property "Manufacturer_Name" "Taoglas" (at 66.04 726.67 0)
+      (effects (font (size 1.27 1.27)) (justify left top) hide)
+    )
+    (property "Manufacturer_Part_Number" "PCB.SMAFRA.HT" (at 66.04 826.67 0)
+      (effects (font (size 1.27 1.27)) (justify left top) hide)
+    )
+    (pin "1")
+    (pin "2")
+    (pin "3")
+    (pin "4")
+    (pin "5")
+    (instances
+      (project "UpDownConverter"
+        (path "/cc9fcf9b-b84f-49ca-8b98-f0ff7034b4a0/89113eb6-a386-4eef-ae89-fc2030098002"
+          (reference "J5") (unit 1)
+        )
+      )
+    )
+  )
+  (symbol (lib_id "power:GND") (at 41.91 46.99 0) (unit 1)
+    (in_bom yes) (on_board yes) (dnp no) (fields_autoplaced)
+    (property "Reference" "#PWR013" (at 41.91 53.34 0)
+      (effects (font (size 1.27 1.27)) hide)
+    )
+    (property "Value" "GND" (at 41.91 52.07 0)
+      (effects (font (size 1.27 1.27)))
+    )
+    (property "Footprint" "" (at 41.91 46.99 0)
+      (effects (font (size 1.27 1.27)) hide)
+    )
+    (property "Datasheet" "" (at 41.91 46.99 0)
+      (effects (font (size 1.27 1.27)) hide)
+    )
+    (pin "1")
+    (instances
+      (project "UpDownConverter"
+        (path "/cc9fcf9b-b84f-49ca-8b98-f0ff7034b4a0/89113eb6-a386-4eef-ae89-fc2030098002"
+          (reference "#PWR013") (unit 1)
+        )
+      )
+    )
+  )
 )
