File: tx_input.kicad_sch (KiCad schematic)
At the start: 0 parts

Commit message: More filter work. Add project title to drawings.
Other:
- company: (none) -> Steves Custom Computers
- title: (none) -> PLUTO RF Card Front-End
Changed lines of the file:
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@@
 (kicad_sch (version 20230121) (generator eeschema)
   (paper "A4")
+  (title_block
+    (title "PLUTO RF Card Front-End")
+    (rev " 001")
+    (company "Steves Custom Computers")
+  )
 )

Commit message: Major restructure. Add power/control busses.
Parts:
- added J2: PCB.SMAFRA.HT, PCBSMAFRAHT, symbol Mouser:PCB.SMAFRA.HT
Connections:
- new net GND: J2.2, J2.3, J2.4, J2.5
- new net TX: J2.1
Other:
- title: PLUTO RF Card Front-End -> PLUTO RF Front-End Card
Changed lines of the file:
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@@
   (paper "A4")
   (title_block
-    (title "PLUTO RF Card Front-End")
+    (title "PLUTO RF Front-End Card")
     (rev " 001")
     (company "Steves Custom Computers")
   )
+  (junction (at 45.72 44.45) (diameter 0) (color 0 0 0 0)
+  )
+  (junction (at 45.72 39.37) (diameter 0) (color 0 0 0 0)
+  )
+  (junction (at 77.47 36.83) (diameter 0) (color 0 0 0 0)
+  )
+  (wire (pts (xy 77.47 36.83) (xy 77.47 44.45))
+    (stroke (width 0) (type default))
+  )
+  (wire (pts (xy 71.12 36.83) (xy 77.47 36.83))
+    (stroke (width 0) (type default))
+  )
+  (wire (pts (xy 45.72 39.37) (xy 50.8 39.37))
+    (stroke (width 0) (type default))
+  )
+  (wire (pts (xy 77.47 34.29) (xy 77.47 36.83))
+    (stroke (width 0) (type default))
+  )
+  (wire (pts (xy 45.72 39.37) (xy 45.72 44.45))
+    (stroke (width 0) (type default))
+  )
+  (wire (pts (xy 77.47 44.45) (xy 45.72 44.45))
+    (stroke (width 0) (type default))
+  )
+  (wire (pts (xy 34.29 34.29) (xy 50.8 34.29))
+    (stroke (width 0) (type default))
+  )
+  (wire (pts (xy 71.12 34.29) (xy 77.47 34.29))
+    (stroke (width 0) (type default))
+  )
+  (wire (pts (xy 50.8 36.83) (xy 45.72 36.83))
+    (stroke (width 0) (type default))
+  )
+  (wire (pts (xy 45.72 36.83) (xy 45.72 39.37))
+    (stroke (width 0) (type default))
+  )
+  (wire (pts (xy 45.72 44.45) (xy 45.72 48.26))
+    (stroke (width 0) (type default))
+  )
+  (hierarchical_label "TX" (shape output) (at 34.29 34.29 180) (fields_autoplaced)
+    (effects (font (size 1.27 1.27)) (justify right))
+  )
+  (symbol (lib_id "power:GND") (at 45.72 48.26 0) (unit 1)
+    (in_bom yes) (on_board yes) (dnp no) (fields_autoplaced)
+    (property "Reference" "#PWR014" (at 45.72 54.61 0)
+      (effects (font (size 1.27 1.27)) hide)
+    )
+    (property "Value" "GND" (at 45.72 53.34 0)
+      (effects (font (size 1.27 1.27)))
+    )
+    (property "Footprint" "" (at 45.72 48.26 0)
+      (effects (font (size 1.27 1.27)) hide)
+    )
+    (property "Datasheet" "" (at 45.72 48.26 0)
+      (effects (font (size 1.27 1.27)) hide)
+    )
+    (pin "1")
+    (instances
+      (project "UpDownConverter"
+        (path "/cc9fcf9b-b84f-49ca-8b98-f0ff7034b4a0/02346fef-99d3-4fce-b956-41e58ea4d527"
+          (reference "#PWR014") (unit 1)
+        )
+      )
+    )
+  )
+  (symbol (lib_id "Mouser:PCB.SMAFRA.HT") (at 50.8 34.29 0) (unit 1)
+    (in_bom yes) (on_board yes) (dnp no) (fields_autoplaced)
+    (property "Reference" "J2" (at 60.96 26.67 0)
+      (effects (font (size 1.27 1.27)))
+    )
+    (property "Value" "PCB.SMAFRA.HT" (at 60.96 29.21 0)
+      (effects (font (size 1.27 1.27)))
+    )
+    (property "Footprint" "PCBSMAFRAHT" (at 67.31 129.21 0)
+      (effects (font (size 1.27 1.27)) (justify left top) hide)
+    )
+    (property "Datasheet" "" (at 67.31 229.21 0)
+      (effects (font (size 1.27 1.27)) (justify left top) hide)
+    )
+    (property "Height" "9" (at 67.31 429.21 0)
+      (effects (font (size 1.27 1.27)) (justify left top) hide)
+    )
+    (property "Mouser Part Number" "960-PCB.SMAFRA.HT" (at 67.31 529.21 0)
+      (effects (font (size 1.27 1.27)) (justify left top) hide)
+    )
+    (property "Mouser Price/Stock" "https://www.mouser.co.uk/ProductDetail/Taoglas/PCB.SMAFRA.HT?qs=RuW%2Fu%252BNMQmubIFYcN8w5Dw%3D%3D" (at 67.31 629.21 0)
+      (effects (font (size 1.27 1.27)) (justify left top) hide)
+    )
+    (property "Manufacturer_Name" "Taoglas" (at 67.31 729.21 0)
+      (effects (font (size 1.27 1.27)) (justify left top) hide)
+    )
+    (property "Manufacturer_Part_Number" "PCB.SMAFRA.HT" (at 67.31 829.21 0)
+      (effects (font (size 1.27 1.27)) (justify left top) hide)
+    )
+    (pin "1")
+    (pin "2")
+    (pin "3")
+    (pin "4")
+    (pin "5")
+    (instances
+      (project "UpDownConverter"
+        (path "/cc9fcf9b-b84f-49ca-8b98-f0ff7034b4a0/02346fef-99d3-4fce-b956-41e58ea4d527"
+          (reference "J2") (unit 1)
+        )
+      )
+    )
+  )
 )
