File: band_select.kicad_sch (KiCad schematic)
At the start: 0 parts

Commit message: More filter work. Add project title to drawings.
Other:
- company: (none) -> Steves Custom Computers
- title: (none) -> PLUTO RF Card Front-End
Changed lines of the file:
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@@
 (kicad_sch (version 20230121) (generator eeschema)
   (paper "A4")
+  (title_block
+    (title "PLUTO RF Card Front-End")
+    (rev " 001")
+    (company "Steves Custom Computers")
+  )
 )

Commit message: Major restructure. Add power/control busses.
Parts:
- added J4: Ctrl Bus Connector, symbol Connector:Conn_01x06_Pin
Connections:
- new net CTRL1: J4.1 (Pin_1)
- new net CTRL2: J4.2 (Pin_2)
- new net CTRL3: J4.3 (Pin_3)
- new net CTRL4: J4.4 (Pin_4)
- new net CTRL5: J4.5 (Pin_5)
- new net CTRL6: J4.6 (Pin_6)
Other:
- title: PLUTO RF Card Front-End -> PLUTO RF Front-End Card
Changed lines of the file:
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@@
   (paper "A4")
   (title_block
-    (title "PLUTO RF Card Front-End")
+    (title "PLUTO RF Front-End Card")
     (rev " 001")
     (company "Steves Custom Computers")
   )
+  (bus_alias "CTRL[1..10]" (members "TR_SEL" "HV_SEL" "UL_SEL" "MIX_SEL" "BAND_SEL[1..2]"))
+  (bus_entry (at 60.96 50.8) (size -2.54 2.54)
+    (stroke (width 0) (type default))
+  )
+  (bus_entry (at 60.96 45.72) (size -2.54 2.54)
+    (stroke (width 0) (type default))
+  )
+  (bus_entry (at 60.96 53.34) (size -2.54 2.54)
+    (stroke (width 0) (type default))
+  )
+  (bus_entry (at 60.96 55.88) (size -2.54 2.54)
+    (stroke (width 0) (type default))
+  )
+  (bus_entry (at 60.96 58.42) (size -2.54 2.54)
+    (stroke (width 0) (type default))
+  )
+  (bus_entry (at 60.96 48.26) (size -2.54 2.54)
+    (stroke (width 0) (type default))
+  )
+  (wire (pts (xy 39.37 60.96) (xy 58.42 60.96))
+    (stroke (width 0) (type default))
+  )
+  (bus (pts (xy 60.96 50.8) (xy 60.96 53.34))
+    (stroke (width 0) (type default))
+  )
+  (bus (pts (xy 60.96 48.26) (xy 60.96 50.8))
+    (stroke (width 0) (type default))
+  )
+  (wire (pts (xy 39.37 53.34) (xy 58.42 53.34))
+    (stroke (width 0) (type default))
+  )
+  (bus (pts (xy 60.96 74.93) (xy 43.18 74.93))
+    (stroke (width 0) (type default))
+  )
+  (bus (pts (xy 60.96 55.88) (xy 60.96 58.42))
+    (stroke (width 0) (type default))
+  )
+  (wire (pts (xy 39.37 48.26) (xy 58.42 48.26))
+    (stroke (width 0) (type default))
+  )
+  (bus (pts (xy 60.96 53.34) (xy 60.96 55.88))
+    (stroke (width 0) (type default))
+  )
+  (bus (pts (xy 60.96 45.72) (xy 60.96 48.26))
+    (stroke (width 0) (type default))
+  )
+  (bus (pts (xy 60.96 58.42) (xy 60.96 74.93))
+    (stroke (width 0) (type default))
+  )
+  (bus (pts (xy 149.86 21.59) (xy 149.86 95.25))
+    (stroke (width 0) (type default))
+  )
+  (bus (pts (xy 43.18 95.25) (xy 149.86 95.25))
+    (stroke (width 0) (type default))
+  )
+  (wire (pts (xy 39.37 50.8) (xy 58.42 50.8))
+    (stroke (width 0) (type default))
+  )
+  (wire (pts (xy 39.37 55.88) (xy 58.42 55.88))
+    (stroke (width 0) (type default))
+  )
+  (wire (pts (xy 39.37 58.42) (xy 58.42 58.42))
+    (stroke (width 0) (type default))
+  )
+  (label "CTRL[1..10]" (at 57.15 74.93 180) (fields_autoplaced)
+    (effects (font (size 1.27 1.27)) (justify right bottom))
+  )
+  (label "CTRL6" (at 39.37 60.96 0)
+    (effects (font (size 1.27 1.27)) (justify left bottom))
+  )
+  (label "CTRL5" (at 39.37 58.42 0) (fields_autoplaced)
+    (effects (font (size 1.27 1.27)) (justify left bottom))
+  )
+  (label "CTRL4" (at 39.37 55.88 0)
+    (effects (font (size 1.27 1.27)) (justify left bottom))
+  )
+  (label "CTRL3" (at 39.37 53.34 0)
+    (effects (font (size 1.27 1.27)) (justify left bottom))
+  )
+  (label "CTRL2" (at 39.37 50.8 0)
+    (effects (font (size 1.27 1.27)) (justify left bottom))
+  )
+  (label "CTRL1" (at 39.37 48.26 0) (fields_autoplaced)
+    (effects (font (size 1.27 1.27)) (justify left bottom))
+  )
+  (hierarchical_label "POWER[1..10]" (shape input) (at 43.18 95.25 180) (fields_autoplaced)
+    (effects (font (size 1.27 1.27)) (justify right))
+  )
+  (hierarchical_label "CTRL[1..10]" (shape output) (at 43.18 74.93 180) (fields_autoplaced)
+    (effects (font (size 1.27 1.27)) (justify right))
+  )
+  (symbol (lib_id "Connector:Conn_01x06_Pin") (at 34.29 53.34 0) (unit 1)
+    (in_bom yes) (on_board yes) (dnp no)
+    (property "Reference" "J4" (at 30.48 35.56 0)
+      (effects (font (size 1.27 1.27)))
+    )
+    (property "Value" "Ctrl Bus Connector" (at 30.48 38.1 0)
+      (effects (font (size 1.27 1.27)))
+    )
+    (property "Footprint" "" (at 34.29 53.34 0)
+      (effects (font (size 1.27 1.27)) hide)
+    )
+    (property "Datasheet" "~" (at 34.29 53.34 0)
+      (effects (font (size 1.27 1.27)) hide)
+    )
+    (pin "1")
+    (pin "2")
+    (pin "3")
+    (pin "4")
+    (pin "5")
+    (pin "6")
+    (instances
+      (project "UpDownConverter"
+        (path "/cc9fcf9b-b84f-49ca-8b98-f0ff7034b4a0/eef86726-0f8f-4e45-83a5-0e3a160b689a"
+          (reference "J4") (unit 1)
+        )
+      )
+    )
+  )
 )
