File: power.kicad_sch (KiCad schematic)
At the start: 0 parts

Commit message: More filter work. Add project title to drawings.
Other:
- company: (none) -> Steves Custom Computers
- title: (none) -> PLUTO RF Card Front-End
Changed lines of the file:
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@@
 (kicad_sch (version 20230121) (generator eeschema)
   (paper "A4")
+  (title_block
+    (title "PLUTO RF Card Front-End")
+    (rev " 001")
+    (company "Steves Custom Computers")
+  )
 )

Commit message: Major restructure. Add power/control busses.
Parts:
- added J1, J6, J7: Conn_01x02_Pin, symbol Connector:Conn_01x02_Pin
Connections:
- new net GND: J1.2 (Pin_2), J6.2 (Pin_2), J7.2 (Pin_2)
- new net POWER1: J1.1 (Pin_1)
- new net POWER2: J6.1 (Pin_1)
- new net POWER3: J7.1 (Pin_1)
Other:
- title: PLUTO RF Card Front-End -> PLUTO RF Front-End Card
Changed lines of the file:
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@@
   (paper "A4")
   (title_block
-    (title "PLUTO RF Card Front-End")
+    (title "PLUTO RF Front-End Card")
     (rev " 001")
     (company "Steves Custom Computers")
   )
+  (bus_entry (at 106.68 86.36) (size -2.54 2.54)
+    (stroke (width 0) (type default))
+  )
+  (bus_entry (at 106.68 49.53) (size -2.54 2.54)
+    (stroke (width 0) (type default))
+  )
+  (bus_entry (at 106.68 67.31) (size -2.54 2.54)
+    (stroke (width 0) (type default))
+  )
+  (wire (pts (xy 62.23 88.9) (xy 104.14 88.9))
+    (stroke (width 0) (type default))
+  )
+  (wire (pts (xy 66.04 95.25) (xy 66.04 91.44))
+    (stroke (width 0) (type default))
+  )
+  (bus (pts (xy 106.68 49.53) (xy 106.68 67.31))
+    (stroke (width 0) (type default))
+  )
+  (wire (pts (xy 60.96 52.07) (xy 104.14 52.07))
+    (stroke (width 0) (type default))
+  )
+  (wire (pts (xy 64.77 54.61) (xy 64.77 58.42))
+    (stroke (width 0) (type default))
+  )
+  (wire (pts (xy 66.04 76.2) (xy 66.04 72.39))
+    (stroke (width 0) (type default))
+  )
+  (wire (pts (xy 66.04 72.39) (xy 62.23 72.39))
+    (stroke (width 0) (type default))
+  )
+  (wire (pts (xy 66.04 91.44) (xy 62.23 91.44))
+    (stroke (width 0) (type default))
+  )
+  (bus (pts (xy 106.68 43.18) (xy 106.68 49.53))
+    (stroke (width 0) (type default))
+  )
+  (wire (pts (xy 62.23 69.85) (xy 104.14 69.85))
+    (stroke (width 0) (type default))
+  )
+  (bus (pts (xy 106.68 172.72) (xy 144.78 172.72))
+    (stroke (width 0) (type default))
+  )
+  (bus (pts (xy 106.68 67.31) (xy 106.68 86.36))
+    (stroke (width 0) (type default))
+  )
+  (bus (pts (xy 106.68 86.36) (xy 106.68 172.72))
+    (stroke (width 0) (type default))
+  )
+  (wire (pts (xy 64.77 54.61) (xy 60.96 54.61))
+    (stroke (width 0) (type default))
+  )
+  (label "POWER1" (at 95.25 52.07 0)
+    (effects (font (size 1.27 1.27)) (justify left bottom))
+  )
+  (label "POWER3" (at 95.25 88.9 0)
+    (effects (font (size 1.27 1.27)) (justify left bottom))
+  )
+  (label "POWER2" (at 96.52 69.85 0)
+    (effects (font (size 1.27 1.27)) (justify left bottom))
+  )
+  (hierarchical_label "POWER[1..10]" (shape output) (at 144.78 172.72 0) (fields_autoplaced)
+    (effects (font (size 1.27 1.27)) (justify left))
+  )
+  (symbol (lib_id "power:GND") (at 66.04 76.2 0) (unit 1)
+    (in_bom yes) (on_board yes) (dnp no) (fields_autoplaced)
+    (property "Reference" "#PWR018" (at 66.04 82.55 0)
+      (effects (font (size 1.27 1.27)) hide)
+    )
+    (property "Value" "GND" (at 66.04 81.28 0)
+      (effects (font (size 1.27 1.27)))
+    )
+    (property "Footprint" "" (at 66.04 76.2 0)
+      (effects (font (size 1.27 1.27)) hide)
+    )
+    (property "Datasheet" "" (at 66.04 76.2 0)
+      (effects (font (size 1.27 1.27)) hide)
+    )
+    (pin "1")
+    (instances
+      (project "UpDownConverter"
+        (path "/cc9fcf9b-b84f-49ca-8b98-f0ff7034b4a0/d983650b-0f6b-433a-9b93-f1b49179bfd3"
+          (reference "#PWR018") (unit 1)
+        )
+      )
+    )
+  )
+  (symbol (lib_id "Connector:Conn_01x02_Pin") (at 55.88 52.07 0) (unit 1)
+    (in_bom yes) (on_board yes) (dnp no) (fields_autoplaced)
+    (property "Reference" "J1" (at 56.515 46.99 0)
+      (effects (font (size 1.27 1.27)))
+    )
+    (property "Value" "Conn_01x02_Pin" (at 56.515 49.53 0)
+      (effects (font (size 1.27 1.27)))
+    )
+    (property "Footprint" "" (at 55.88 52.07 0)
+      (effects (font (size 1.27 1.27)) hide)
+    )
+    (property "Datasheet" "~" (at 55.88 52.07 0)
+      (effects (font (size 1.27 1.27)) hide)
+    )
+    (pin "1")
+    (pin "2")
+    (instances
+      (project "UpDownConverter"
+        (path "/cc9fcf9b-b84f-49ca-8b98-f0ff7034b4a0/d983650b-0f6b-433a-9b93-f1b49179bfd3"
+          (reference "J1") (unit 1)
+        )
+      )
+    )
+  )
+  (symbol (lib_id "power:GND") (at 66.04 95.25 0) (unit 1)
+    (in_bom yes) (on_board yes) (dnp no) (fields_autoplaced)
+    (property "Reference" "#PWR019" (at 66.04 101.6 0)
+      (effects (font (size 1.27 1.27)) hide)
+    )
+    (property "Value" "GND" (at 66.04 100.33 0)
+      (effects (font (size 1.27 1.27)))
+    )
+    (property "Footprint" "" (at 66.04 95.25 0)
+      (effects (font (size 1.27 1.27)) hide)
+    )
+    (property "Datasheet" "" (at 66.04 95.25 0)
+      (effects (font (size 1.27 1.27)) hide)
+    )
+    (pin "1")
+    (instances
+      (project "UpDownConverter"
+        (path "/cc9fcf9b-b84f-49ca-8b98-f0ff7034b4a0/d983650b-0f6b-433a-9b93-f1b49179bfd3"
+          (reference "#PWR019") (unit 1)
+        )
+      )
+    )
+  )
+  (symbol (lib_id "power:GND") (at 64.77 58.42 0) (unit 1)
+    (in_bom yes) (on_board yes) (dnp no) (fields_autoplaced)
+    (property "Reference" "#PWR02" (at 64.77 64.77 0)
+      (effects (font (size 1.27 1.27)) hide)
+    )
+    (property "Value" "GND" (at 64.77 63.5 0)
+      (effects (font (size 1.27 1.27)))
+    )
+    (property "Footprint" "" (at 64.77 58.42 0)
+      (effects (font (size 1.27 1.27)) hide)
+    )
+    (property "Datasheet" "" (at 64.77 58.42 0)
+      (effects (font (size 1.27 1.27)) hide)
+    )
+    (pin "1")
+    (instances
+      (project "UpDownConverter"
+        (path "/cc9fcf9b-b84f-49ca-8b98-f0ff7034b4a0/d983650b-0f6b-433a-9b93-f1b49179bfd3"
+          (reference "#PWR02") (unit 1)
+        )
+      )
+    )
+  )
+  (symbol (lib_id "Connector:Conn_01x02_Pin") (at 57.15 69.85 0) (unit 1)
+    (in_bom yes) (on_board yes) (dnp no) (fields_autoplaced)
+    (property "Reference" "J6" (at 57.785 64.77 0)
+      (effects (font (size 1.27 1.27)))
+    )
+    (property "Value" "Conn_01x02_Pin" (at 57.785 67.31 0)
+      (effects (font (size 1.27 1.27)))
+    )
+    (property "Footprint" "" (at 57.15 69.85 0)
+      (effects (font (size 1.27 1.27)) hide)
+    )
+    (property "Datasheet" "~" (at 57.15 69.85 0)
+      (effects (font (size 1.27 1.27)) hide)
+    )
+    (pin "1")
+    (pin "2")
+    (instances
+      (project "UpDownConverter"
+        (path "/cc9fcf9b-b84f-49ca-8b98-f0ff7034b4a0/d983650b-0f6b-433a-9b93-f1b49179bfd3"
+          (reference "J6") (unit 1)
+        )
+      )
+    )
+  )
+  (symbol (lib_id "Connector:Conn_01x02_Pin") (at 57.15 88.9 0) (unit 1)
+    (in_bom yes) (on_board yes) (dnp no) (fields_autoplaced)
+    (property "Reference" "J7" (at 57.785 83.82 0)
+      (effects (font (size 1.27 1.27)))
+    )
+    (property "Value" "Conn_01x02_Pin" (at 57.785 86.36 0)
+      (effects (font (size 1.27 1.27)))
+    )
+    (property "Footprint" "" (at 57.15 88.9 0)
+      (effects (font (size 1.27 1.27)) hide)
+    )
+    (property "Datasheet" "~" (at 57.15 88.9 0)
+      (effects (font (size 1.27 1.27)) hide)
+    )
+    (pin "1")
+    (pin "2")
+    (instances
+      (project "UpDownConverter"
+        (path "/cc9fcf9b-b84f-49ca-8b98-f0ff7034b4a0/d983650b-0f6b-433a-9b93-f1b49179bfd3"
+          (reference "J7") (unit 1)
+        )
+      )
+    )
+  )
 )
